File: posey-wx.kicad_sch (KiCad schematic)
At the start: 29 parts, among them J1 TC2050-IDC-NL, Y1 XTAL, Y2 XTAL

Commit message: w2310 µ380
Parts:
- removed µC1: uC BMD-350-A-R, posey:BMD-350-A-R, symbol posey:uC BMD-350-A-R
- added U1: BMD-380-A-R, posey:XCVR_BMD-380-A-R, symbol posey:BMD-380-A-R
Connections:
- net GND: now also U1.1 (GND), U1.2 (GND), U1.23 (GND), U1.3 (GND), U1.35 (GND), U1.5 (GND), U1.54 (GND), U1.55 (GND), U1.56 (GND), U1.57 (GND), U1.58 (GND), U1.63 (GND)
- net IMU_nINT: now also U1.33 (P0.26)
- net IMU_nRESET: now also U1.34 (P0.04/AIN2)
- net I_CHG: now also U1.31 (P0.05/AIN3)
- net SCL/SPI_SCK: now also U1.28 (P1.09/TRACEDATA[3])
- net SDA/SPI_CIPO: now also U1.26 (P0.12/TRACEDATA[1])
- net SPI_COPI: now also U1.32 (P0.27)
- net SPI_CS_IMU: now also U1.30 (P0.06)
- net SWCLK: now also U1.4 (SWCLK)
- net SWDIO: now also U1.7 (SWDIO)
- net SWO: now also U1.11 (P1.00/TRACEDATA[0]/SWO)
- net VCC: now also U1.22 (VCCH), U1.24 (VCC)
- net nRESET: now also U1.12 (P0.18/RESET)
- net VBAT_SENSE: now reaches R11.1, R9.2
- net VBAT_SENSE: now also U1.43 (P0.28/AIN4)
- net at C8.2, Y1.1: now also U1.38 (P0.00/XTAL1)
- net at C9.2, Y1.2: now also U1.36 (P0.01/XTAL2)
- net EXT_P0_12 renamed EXT_P0_11
- net EXT_P0_11: now also U1.18 (P0.11/TRACEDATA[2])
- net EXT_P0_15 renamed EXT_P0_14
- net EXT_P0_14: now also U1.16 (P0.14)
Other:
- moved on the sheet: C8, C9, Y1

Commit message: Updated readme, license, and version.
Parts:
- added C10: 0.1µ, Capacitor_SMD:C_0402_1005Metric, symbol Device:C
- added J2: Conn_02x06_Odd_Even, Connector_PinHeader_1.27mm:PinHeader_2x06_P1.27mm_Vertical, symbol Connector_Generic:Conn_02x06_Odd_Even
- IMU1: value BNO080 -> BNO086
Connections:
- net GND: now also C10.2, J2.7 (Pin_7), J2.9 (Pin_9); no longer IMU1.5 (PS1), IMU1.6 (PS0/WAKE)
- net IMU_nINT: now also J2.3 (Pin_3)
- net IMU_nRESET: now also J2.2 (Pin_2)
- net SCL/SPI_SCK: now also J2.12 (Pin_12)
- net SDA/SPI_CIPO: now also J2.10 (Pin_10)
- net SPI_COPI: now also J2.6 (Pin_6)
- net SPI_CS_IMU: now also J2.8 (Pin_8)
- net VBAT: now also J2.11 (Pin_11)
- net VCC: now also C10.1, J2.1 (Pin_1)
- net IMU_PS1: now reaches U1.42 (P0.30/AIN6)
- net IMU_PS1: now also IMU1.5 (PS1), J2.4 (Pin_4)
- net IMU_PS0: now reaches U1.45 (P1.14)
- net IMU_PS0: now also IMU1.6 (PS0/WAKE), J2.5 (Pin_5)
Other:
- note removed: "2023.10.18"
- note removed: "2310"
- note removed: "Posey IMU Platform"
- note removed: "Soft Machines Lab Carnegie Mellon University License here"
- company: (none) -> Soft Machines Lab
- title: (none) -> Posey Watch
